Commit message: update

File: schunk_svh_description/urdf/svh-include.urdf.xacro (robot description, xacro)
@@ -2,5 +2,5 @@
 <robot name="svh" xmlns:xacro="http://www.ros.org/wiki/xacro">
   <xacro:include filename="$(find schunk_svh_description)/urdf/svh.urdf.xacro" />
-  <xacro:property name="left_right" default="left_hand" />
+  <xacro:property name="left_right" default="left" />
   <!-- <link name="world" />
   <joint name="world_joint" type="fixed">
@@ -9,14 +9,15 @@
     <origin rpy="0.0 0.0 0.0" xyz="0.0 0.0 0.0" />
   </joint> -->
-  <link name="base_link" />
-  <xacro:if value="${left_right == 'left_hand'}">
+  <xacro:if value="${left_right == 'left'}">
     <xacro:arg name="name_prefix" default="left_hand"/>
-    <xacro:svh parent="base_link" name="$(arg name_prefix)" side="-1">
+    <link name="${left_right}_base_link" />
+    <xacro:svh parent="${left_right}_base_link" name="$(arg name_prefix)" side="-1">
       <origin xyz="0 0 0" rpy="0 0 0" />
     </xacro:svh>
   </xacro:if>
-  <xacro:if value="${left_right == 'right_hand'}">
+  <xacro:if value="${left_right == 'right'}">
     <xacro:arg name="name_prefix" default="right_hand"/>
-    <xacro:svh parent="base_link" name="$(arg name_prefix)" side="1">
+    <link name="${left_right}_base_link" />
+    <xacro:svh parent="${left_right}_base_link" name="$(arg name_prefix)" side="1">
       <origin xyz="0 0 0" rpy="0 0 0" />
     </xacro:svh>

File: schunk_svh_description/urdf/svh.urdf.xacro (robot description, xacro)
@@ -8,5 +8,5 @@
     <!-- RIGHT HAND = 1, LEFT HAND = -1 -->
     <!-- BASE_LINE LINKS -->
-    <joint name="${name}_base_joint" type="fixed" >
+    <joint name="${name}_base_joint" type="fixed">
       <xacro:insert_block name="origin" />
       <parent link="${parent}" />
@@ -19,5 +19,5 @@
         <geometry>
           <mesh filename="package://schunk_svh_description/meshes/base10.dae" />
-	</geometry>
+        </geometry>
       </visual>
       <collision>
@@ -25,9 +25,9 @@
         <geometry>
           <mesh filename="package://schunk_svh_description/meshes/base10.dae" />
-	</geometry>
-      </collision>
-      <inertial>
-        <mass value="0.57743"/>
-        <origin xyz="0.0 -2.3e-05 0.139371"/>
+        </geometry>
+      </collision>
+      <inertial>
+        <mass value="0.57743" />
+        <origin xyz="0.0 -2.3e-05 0.139371" />
         <inertia ixx="0.04725" ixy="-0.0" ixz="-0.0" iyy="0.04717" iyz="0.0" izz="0.07606" />
       </inertial>
@@ -40,5 +40,5 @@
       <!-- 	<material name="${name}_green" /> -->
       <!-- </visual> -->
-      <xacro:default_inertial mass="0.01"/>
+      <xacro:default_inertial mass="0.01" />
     </link>
     <link name="${name}_h">
@@ -50,5 +50,5 @@
       <!-- 	<material name="${name}_green" /> -->
       <!-- </visual> -->
-      <xacro:default_inertial mass="0.01"/>
+      <xacro:default_inertial mass="0.01" />
     </link>
     <link name="${name}_d2">
@@ -60,40 +60,40 @@
       <!-- 	<material name="${name}_green" /> -->
       <!-- </visual> -->
-      <xacro:default_inertial mass="0.01"/>
+      <xacro:default_inertial mass="0.01" />
     </link>
     <!-- LENGTH NOT FOUND IN DATASHEET! GUESSED!!! -->
     <link name="${name}_e1">
       <visual>
-	<origin rpy="0 0 0" xyz="0 0.01313 0" />
-	<geometry>
+        <origin rpy="0 0 0" xyz="0 0.01313 0" />
+        <geometry>
           <mesh scale="${side*(1)} 1 1" filename="package://schunk_svh_description/meshes/h10.dae" />
-	</geometry>
-      </visual>
-      <collision>
-	<origin rpy="0 0 0" xyz="0 0.01313 0" />
-	<geometry>
+        </geometry>
+      </visual>
+      <collision>
+        <origin rpy="0 0 0" xyz="0 0.01313 0" />
+        <geometry>
           <mesh scale="${side*(1)} 1 1" filename="package://schunk_svh_description/meshes/h10.dae" />
-	</geometry>
-      </collision>
-      <xacro:default_inertial mass="0.01"/>
+        </geometry>
+      </collision>
+      <xacro:default_inertial mass="0.01" />
     </link>
     <!-- LENGTH NOT FOUND IN DATASHEET! GUESSED!!! -->
     <link name="${name}_e2">
       <visual>
-	<origin xyz="${side*(-0.0007)} 0 -0.01002" />
-	<geometry>
+        <origin xyz="${side*(-0.0007)} 0 -0.01002" />
+        <geometry>
           <mesh scale="${side*(1)} 1 1" filename="package://schunk_svh_description/meshes/h11.dae" />
-	</geometry>
-      </visual>
-      <collision>
-	<origin xyz="${side*(-0.0007)} 0 -0.01002" />
-	<geometry>
+        </geometry>
+      </visual>
+      <collision>
+        <origin xyz="${side*(-0.0007)} 0 -0.01002" />
+        <geometry>
           <mesh scale="${side*(1)} 1 1" filename="package://schunk_svh_description/meshes/h11.dae" />
-	</geometry>
-      </collision>
-      <inertial>
-        <mass value="0.46184"/>
-        <origin xyz="0.145071 -0.037868 0.323449"/>
-        <inertia ixx="0.01908" ixy="-0.00121" ixz="-0.00011" iyy="0.01704" iyz="0.00277" izz="0.00862"/>
+        </geometry>
+      </collision>
+      <inertial>
+        <mass value="0.46184" />
+        <origin xyz="0.145071 -0.037868 0.323449" />
+        <inertia ixx="0.01908" ixy="-0.00121" ixz="-0.00011" iyy="0.01704" iyz="0.00277" izz="0.00862" />
       </inertial>
     </link>
@@ -107,8 +107,7 @@
       <!-- 	<material name="green" /> -->
       <!-- </visual> -->
-      <xacro:default_inertial mass="0.01"/>
-    </link>
-    <link name="${name}_e">
-    </link>
+      <xacro:default_inertial mass="0.01" />
+    </link>
+    <link name="${name}_e"></link>
     <!-- LENGTH NOT FOUND IN DATASHEET! GUESSED, BUT POSITION CALCULATED: E4 = D-G-F!!! -->
     <link name="${name}_e4">
@@ -120,5 +119,5 @@
       <!-- 	<material name="green" /> -->
       <!-- </visual> -->
-      <xacro:default_inertial mass="0.01"/>
+      <xacro:default_inertial mass="0.01" />
     </link>
     <!-- LENGTH NOT FOUND IN DATASHEET! GUESSED, BUT POSITION CALCULATED: E5 = D-G!!! -->
@@ -131,78 +130,78 @@
       <!-- 	<material name="green" /> -->
       <!-- </visual> -->
-      <xacro:default_inertial mass="0.01"/>
+      <xacro:default_inertial mass="0.01" />
     </link>
     <!-- THUMB LINKS -->
     <link name="${name}_z">
       <visual>
-	<origin xyz="0 0 0.02442" />
-	<geometry>
+        <origin xyz="0 0 0.02442" />
+        <geometry>
           <mesh scale="1 ${side*(1)} 1" filename="package://schunk_svh_description/meshes/d10.dae" />
-	</geometry>
-      </visual>
-      <collision>
-	<origin xyz="0 0 0.02442" />
-	<geometry>
+        </geometry>
+      </visual>
+      <collision>
+        <origin xyz="0 0 0.02442" />
+        <geometry>
           <mesh scale="1 ${side*(1)} 1" filename="package://schunk_svh_description/meshes/d10.dae" />
-	</geometry>
-      </collision>
-      <inertial>
-        <mass value="0.0739"/>
-        <origin xyz="0.0 0.002024 0.178636"/>
-        <inertia ixx="0.00103" ixy="-0.0" ixz="-0.0" iyy="0.00165" iyz="4e-05" izz="0.00111"/>
+        </geometry>
+      </collision>
+      <inertial>
+        <mass value="0.0739" />
+        <origin xyz="0.0 0.002024 0.178636" />
+        <inertia ixx="0.00103" ixy="-0.0" ixz="-0.0" iyy="0.00165" iyz="4e-05" izz="0.00111" />
       </inertial>
     </link>
     <link name="${name}_virtual_a">
-      <xacro:default_inertial mass="0.01"/>
+      <xacro:default_inertial mass="0.01" />
     </link>
     <link name="${name}_a">
       <visual>
-	<geometry>
+        <geometry>
           <mesh scale="1 ${side*(1)} ${side*(1)}" filename="package://schunk_svh_description/meshes/d11.dae" />
-	</geometry>
-      </visual>
-      <collision>
-	<geometry>
+        </geometry>
+      </visual>
+      <collision>
+        <geometry>
           <mesh scale="1 ${side*(1)} ${side*(1)}" filename="package://schunk_svh_description/meshes/d11.dae" />
-	</geometry>
-      </collision>
-      <inertial>
-        <mass value="0.41222"/>
-        <origin xyz="0.240205 0.010733 0.00019"/>
-        <inertia ixx="0.00413" ixy="0.00073" ixz="-0.0" iyy="0.01679" iyz="0.0" izz="0.01796"/>
+        </geometry>
+      </collision>
+      <inertial>
+        <mass value="0.41222" />
+        <origin xyz="0.240205 0.010733 0.00019" />
+        <inertia ixx="0.00413" ixy="0.00073" ixz="-0.0" iyy="0.01679" iyz="0.0" izz="0.01796" />
       </inertial>
     </link>
     <link name="${name}_b">
       <visual>
-	<geometry>
+        <geometry>
           <mesh scale="1 ${side*(1)} ${side*(1)}" filename="package://schunk_svh_description/meshes/d12.dae" />
-	</geometry>
-      </visual>
-      <collision>
-	<geometry>
+        </geometry>
+      </visual>
+      <collision>
+        <geometry>
           <mesh scale="1 ${side*(1)} ${side*(1)}" filename="package://schunk_svh_description/meshes/d12.dae" />
-	</geometry>
-      </collision>
-      <inertial>
-        <mass value="0.08224"/>
-        <origin xyz="0.123157 -0.008382 -2.7e-05"/>
-        <inertia ixx="0.00089" ixy="5e-05" ixz="0.0" iyy="0.00139" iyz="0.0" izz="0.00103"/>
+        </geometry>
+      </collision>
+      <inertial>
+        <mass value="0.08224" />
+        <origin xyz="0.123157 -0.008382 -2.7e-05" />
+        <inertia ixx="0.00089" ixy="5e-05" ixz="0.0" iyy="0.00139" iyz="0.0" izz="0.00103" />
       </inertial>
     </link>
     <link name="${name}_c">
       <visual>
-	<geometry>
+        <geometry>
           <mesh scale="1 ${side*(1)} ${side*(1)}" filename="package://schunk_svh_description/meshes/d13.dae" />
-	</geometry>
-      </visual>
-      <collision>
-	<geometry>
+        </geometry>
+      </visual>
+      <collision>
+        <geometry>
           <mesh scale="1 ${side*(1)} ${side*(1)}" filename="package://schunk_svh_description/meshes/d13.dae" />
-	</geometry>
-      </collision>
-      <inertial>
-        <mass value="0.06198"/>
-        <origin xyz="0.113729 0.01094 0.0"/>
-        <inertia ixx="0.00025" ixy="-0.0" ixz="-0.0" iyy="0.00051" iyz="0.0" izz="0.00052"/>
+        </geometry>
+      </collision>
+      <inertial>
+        <mass value="0.06198" />
+        <origin xyz="0.113729 0.01094 0.0" />
+        <inertia ixx="0.00025" ixy="-0.0" ixz="-0.0" iyy="0.00051" iyz="0.0" izz="0.00052" />
       </inertial>
     </link>
@@ -210,70 +209,70 @@
     <link name="${name}_virtual_l">
       <visual>
-	<origin xyz="0 0 0.01321" />
-	<geometry>
+        <origin xyz="0 0 0.01321" />
+        <geometry>
           <mesh filename="package://schunk_svh_description/meshes/f10.dae" />
-	</geometry>
-      </visual>
-      <collision>
-	<origin xyz="0 0 0.01321" />
-	<geometry>
+        </geometry>
+      </visual>
+      <collision>
+        <origin xyz="0 0 0.01321" />
+        <geometry>
           <mesh filename="package://schunk_svh_description/meshes/f10.dae" />
-	</geometry>
-      </collision>
-      <inertial>
-        <mass value="0.02383"/>
-        <origin xyz="0.003634 0.000206 -0.09885"/>
-        <inertia ixx="0.00021" ixy="-0.0" ixz="-1e-05" iyy="0.00011" iyz="-0.0" izz="0.00019"/>
+        </geometry>
+      </collision>
+      <inertial>
+        <mass value="0.02383" />
+        <origin xyz="0.003634 0.000206 -0.09885" />
+        <inertia ixx="0.00021" ixy="-0.0" ixz="-1e-05" iyy="0.00011" iyz="-0.0" izz="0.00019" />
       </inertial>
     </link>
     <link name="${name}_l">
       <visual>
-	<geometry>
+        <geometry>
           <mesh filename="package://schunk_svh_description/meshes/f11.dae" />
-	</geometry>
-      </visual>
-      <collision>
-	<geometry>
+        </geometry>
+      </visual>
+      <collision>
+        <geometry>
           <mesh filename="package://schunk_svh_description/meshes/f11.dae" />
-	</geometry>
-      </collision>
-      <inertial>
-        <mass value="0.13003"/>
-        <origin xyz="0.261673 0.003521 0.0"/>
-        <inertia ixx="0.00051" ixy="-3e-05" ixz="0.0" iyy="0.00335" iyz="-0.0" izz="0.00344"/>
+        </geometry>
+      </collision>
+      <inertial>
+        <mass value="0.13003" />
+        <origin xyz="0.261673 0.003521 0.0" />
+        <inertia ixx="0.00051" ixy="-3e-05" ixz="0.0" iyy="0.00335" iyz="-0.0" izz="0.00344" />
       </inertial>
     </link>
     <link name="${name}_p">
       <visual>
-	<geometry>
+        <geometry>
           <mesh filename="package://schunk_svh_description/meshes/f12.dae" />
-	</geometry>
-      </visual>
-      <collision>
-	<geometry>
+        </geometry>
+      </visual>
+      <collision>
+        <geometry>
           <mesh filename="package://schunk_svh_description/meshes/f12.dae" />
-	</geometry>
-      </collision>
-      <inertial>
-        <mass value="0.03264"/>
-        <origin xyz="0.1384 -0.004609 0.0"/>
-        <inertia ixx="0.00016" ixy="-0.0" ixz="0.0" iyy="0.00031" iyz="-0.0" izz="0.00024"/>
+        </geometry>
+      </collision>
+      <inertial>
+        <mass value="0.03264" />
+        <origin xyz="0.1384 -0.004609 0.0" />
+        <inertia ixx="0.00016" ixy="-0.0" ixz="0.0" iyy="0.00031" iyz="-0.0" izz="0.00024" />
       </inertial>
     </link>
     <link name="${name}_t">
       <visual>
-	<geometry>
+        <geometry>
           <mesh filename="package://schunk_svh_description/meshes/f13.dae" />
-	</geometry>
-      </visual>
-      <collision>
-	<geometry>
+        </geometry>
+      </visual>
+      <collision>
+        <geometry>
           <mesh filename="package://schunk_svh_description/meshes/f13.dae" />
-	</geometry>
-      </collision>
-      <inertial>
-        <mass value="0.0324"/>
-        <origin xyz="0.102924 0.000592 0.0"/>
-        <inertia ixx="9e-05" ixy="-1e-05" ixz="-0.0" iyy="0.00017" iyz="0.0" izz="0.00017"/>
+        </geometry>
+      </collision>
+      <inertial>
+        <mass value="0.0324" />
+        <origin xyz="0.102924 0.000592 0.0" />
+        <inertia ixx="9e-05" ixy="-1e-05" ixz="-0.0" iyy="0.00017" iyz="0.0" izz="0.00017" />
       </inertial>
     </link>
@@ -281,70 +280,70 @@
     <link name="${name}_virtual_k">
       <visual>
-	<origin xyz="0 0 0.01321" />
-	<geometry>
+        <origin xyz="0 0 0.01321" />
+        <geometry>
           <mesh filename="package://schunk_svh_description/meshes/f20.dae" />
-	</geometry>
-      </visual>
-      <collision>
-	<origin xyz="0 0 0.01321" />
-	<geometry>
+        </geometry>
+      </visual>
+      <collision>
+        <origin xyz="0 0 0.01321" />
+        <geometry>
           <mesh filename="package://schunk_svh_description/meshes/f20.dae" />
-	</geometry>
-      </collision>
-      <inertial>
-        <mass value="0.02377"/>
-        <origin xyz="0.003357 -8e-06 -0.099643"/>
-        <inertia ixx="0.00021" ixy="-0.0" ixz="-1e-05" iyy="0.00011" iyz="0.0" izz="0.00019"/>
+        </geometry>
+      </collision>
+      <inertial>
+        <mass value="0.02377" />
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