Commit message: Adding bias at robot_state and custom state publisher

File: schunk_svh_description/urdf/svh.urdf.xacro (robot description, xacro)
@@ -565,5 +565,5 @@
       <child link="${name}_b" />
       <limit effort="1000.0" lower="0.0" upper="0.98506" velocity="1" />
-      <origin xyz="0.0485 0 0" rpy="0 0 0" />
+      <origin xyz="0.0485 0 0" rpy="0 0 ${side*(0.2)}" />
       <axis xyz="0 0 ${side*(1)}" />
       <mimic joint="${name}_Thumb_Flexion" multiplier="1.01511" offset="0" />
@@ -582,5 +582,5 @@
       <child link="${name}_p" />
       <limit effort="1000.0" lower="0" upper="1.334" velocity="1" />
-      <origin xyz="0.04804 0 0" rpy="0 0 0" />
+      <origin xyz="0.04804 0 0" rpy="0 0 0.25" />
       <axis xyz="0 0 1" />
     </joint>
@@ -589,5 +589,5 @@
       <child link="${name}_l" />
       <limit effort="1000.0" lower="0.0" upper="0.79849" velocity="1" />
-      <origin xyz="0 0 0" rpy="-1.5707 0 0" />
+      <origin xyz="0 0 0" rpy="-1.5707 0 0.0" />
       <axis xyz="0 0 1" />
     </joint>
@@ -606,5 +606,5 @@
       <child link="${name}_k" />
       <limit effort="1000.0" lower="0.0" upper="0.79849" velocity="1" />
-      <origin xyz="0 0 0" rpy="-1.5707 0 0" />
+      <origin xyz="0 0 0" rpy="-1.5707 0 0.0" />
       <axis xyz="0 0 1" />
     </joint>
@@ -613,5 +613,5 @@
       <child link="${name}_o" />
       <limit effort="1000.0" lower="0" upper="1.334" velocity="1" />
-      <origin xyz="0.05004 0 0" rpy="0 0 0" />
+      <origin xyz="0.05004 0 0" rpy="0 0 0.25" />
       <axis xyz="0 0 1" />
     </joint>
@@ -620,5 +620,5 @@
       <child link="${name}_s" />
       <limit effort="1000.0" lower="0" upper="1.334" velocity="1" />
-      <origin xyz="0.032 0 0" rpy="0 0 0" />
+      <origin xyz="0.032 0 0" rpy="0 0 0.25" />
       <axis xyz="0 0 1" />
       <mimic joint="${name}_Middle_Finger_Distal" multiplier="1.0454" offset="0" />
@@ -636,5 +636,5 @@
       <child link="${name}_n" />
       <limit effort="1000.0" lower="0" upper="1.334" velocity="1" />
-      <origin xyz="0.05004 0 0" rpy="0 0 0" />
+      <origin xyz="0.05004 0 0" rpy="0 0 0.3" />
       <axis xyz="0 0 1" />
       <mimic joint="${name}_Ring_Finger" multiplier="1.3588" offset="0" />
@@ -644,5 +644,5 @@
       <child link="${name}_r" />
       <limit effort="1000.0" lower="0" upper="1.395" velocity="1" />
-      <origin xyz="0.032 0 0" rpy="0 0 0" />
+      <origin xyz="0.032 0 0" rpy="0 0 0.3" />
       <axis xyz="0 0 1" />
       <mimic joint="${name}_Ring_Finger" multiplier="1.42093" offset="0" />
@@ -660,5 +660,5 @@
       <child link="${name}_m" />
       <limit effort="1000.0" lower="0" upper="1.334" velocity="1" />
-      <origin xyz="0.04454 0 0" rpy="0 0 0" />
+      <origin xyz="0.04454 0 0" rpy="0 0 0.3" />
       <axis xyz="0 0 1" />
       <mimic joint="${name}_Pinky" multiplier="1.35880" offset="0" />
@@ -668,5 +668,5 @@
       <child link="${name}_q" />
       <limit effort="1000.0" lower="0" upper="1.3971" velocity="1" />
-      <origin xyz="0.022 0 0" rpy="0 0 0" />
+      <origin xyz="0.022 0 0" rpy="0 0 0.3" />
       <axis xyz="0 0 1" />
       <mimic joint="${name}_Pinky" multiplier="1.42307" offset="0" />
